File: Hardware/Kicad_Project/MASA_Rover_1.0/DCmotorExt.kicad_sch (KiCad schematic)
At the start: 45 parts, among them J39 Screw_Terminal_01x01, J40 Screw_Terminal_01x01, J41 Screw_Terminal_01x01, J42 Screw_Terminal_01x01, J43 Screw_Terminal_01x01, J44 Screw_Terminal_01x01, J45 Screw_Terminal_01x01, J46 Screw_Terminal_01x01, J47 Screw_Terminal_01x01, U16 DRV8876,16-HTSSOP, U17 DRV8876,16-HTSSOP, U18 DRV8876,16-HTSSOP, U19 DRV8876,16-HTSSOP

Commit message: update hardware
Connections:
- net +3.3V renamed +3V3
