File: Hardware/Kicad_Project/MASA_Rover_1.0/I2CExpender.kicad_sch (KiCad schematic)
At the start: 18 parts, among them J6 Conn_01x04, J7 Conn_02x10_Top_Bottom, U4 MAX11603EEE+, U5 PCA9535D, U6 PCA9685PW_112

Commit message: update hardware
Connections:
- net PWM0: now also J7.7 (Pin_7)
- net PWM1: now also J7.5 (Pin_5)
- net PWM12: no longer J7.1 (Pin_1)
- net PWM13: no longer J7.3 (Pin_3)
- net PWM14: no longer J7.5 (Pin_5)
- net PWM15: no longer J7.7 (Pin_7)
- net PWM2: now also J7.3 (Pin_3)
- net PWM3: now also J7.1 (Pin_1)
Changed lines of the file:
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@@
+    (stroke (width 0) (type default) (color 0 0 0 0))
+  )
+  (wire (pts (xy 144.78 116.84) (xy 152.4 116.84))
     (stroke (width 0) (type default) (color 0 0 0 0))
   )
@@
     (stroke (width 0) (type default) (color 0 0 0 0))
   )
-  (wire (pts (xy 144.78 116.84) (xy 152.4 116.84))
-    (stroke (width 0) (type default) (color 0 0 0 0))
-  )
   (wire (pts (xy 25.4 127) (xy 25.4 97.79))
     (stroke (width 0) (type default) (color 0 0 0 0))
@@
     (stroke (width 0) (type default) (color 0 0 0 0))
   )
+  (wire (pts (xy 144.78 119.38) (xy 152.4 119.38))
+    (stroke (width 0) (type default) (color 0 0 0 0))
+  )
   (wire (pts (xy 72.39 115.57) (xy 81.28 115.57))
     (stroke (width 0) (type default) (color 0 0 0 0))
@@
   )
   (wire (pts (xy 49.53 102.87) (xy 45.72 102.87))
-    (stroke (width 0) (type default) (color 0 0 0 0))
-  )
-  (wire (pts (xy 144.78 119.38) (xy 152.4 119.38))
     (stroke (width 0) (type default) (color 0 0 0 0))
   )
@@
     (effects (font (size 1.27 1.27)) (justify right bottom))
   )
-  (label "IO1_3" (at 199.39 144.78 0)
+  (label "IO1_3" (at 199.39 119.38 0)
     (effects (font (size 1.27 1.27)) (justify left bottom))
   )
@@
     (effects (font (size 1.27 1.27)) (justify right bottom))
   )
-  (label "IO0_0" (at 199.39 119.38 0)
-    (effects (font (size 1.27 1.27)) (justify left bottom))
-  )
-  (label "PWM9" (at 199.39 64.77 0)
+  (label "IO0_0" (at 199.39 138.43 0)
+    (effects (font (size 1.27 1.27)) (justify left bottom))
+  )
+  (label "PWM5" (at 199.39 64.77 0)
     (effects (font (size 1.27 1.27)) (justify left bottom))
   )
@@
     (effects (font (size 1.27 1.27)) (justify right bottom))
   )
-  (label "PWM13" (at 77.47 166.37 0)
-    (effects (font (size 1.27 1.27)) (justify left bottom))
-  )
   (label "IO1_2" (at 152.4 121.92 180)
     (effects (font (size 1.27 1.27)) (justify right bottom))
@@
     (effects (font (size 1.27 1.27)) (justify right bottom))
   )
-  (label "PWM11" (at 199.39 69.85 0)
+  (label "PWM7" (at 199.39 69.85 0)
     (effects (font (size 1.27 1.27)) (justify left bottom))
   )
@@
     (effects (font (size 1.27 1.27)) (justify right bottom))
   )
-  (label "PWM5" (at 199.39 99.06 0)
+  (label "PWM12" (at 199.39 99.06 0)
     (effects (font (size 1.27 1.27)) (justify left bottom))
   )
@@
     (effects (font (size 1.27 1.27)) (justify right bottom))
   )
-  (label "PWM1" (at 199.39 86.36 0)
+  (label "PWM8" (at 199.39 86.36 0)
     (effects (font (size 1.27 1.27)) (justify left bottom))
   )
@@
     (effects (font (size 1.27 1.27)) (justify left bottom))
   )
-  (label "IO1_4" (at 199.39 147.32 0)
+  (label "IO1_4" (at 199.39 121.92 0)
     (effects (font (size 1.27 1.27)) (justify left bottom))
   )
@@
     (effects (font (size 1.27 1.27)) (justify right bottom))
   )
-  (label "IO0_2" (at 199.39 125.73 0)
+  (label "IO0_2" (at 199.39 147.32 0)
     (effects (font (size 1.27 1.27)) (justify left bottom))
   )
@@
     (effects (font (size 1.27 1.27)) (justify right bottom))
   )
+  (label "PWM2" (at 77.47 166.37 0)
+    (effects (font (size 1.27 1.27)) (justify left bottom))
+  )
   (label "IO0_2" (at 152.4 101.6 180)
     (effects (font (size 1.27 1.27)) (justify right bottom))
   )
-  (label "PWM0" (at 199.39 83.82 0)
+  (label "PWM9" (at 199.39 83.82 0)
     (effects (font (size 1.27 1.27)) (justify left bottom))
   )
@@
     (effects (font (size 1.27 1.27)) (justify right bottom))
   )
-  (label "IO1_2" (at 199.39 142.24 0)
+  (label "IO1_2" (at 199.39 130.81 0)
     (effects (font (size 1.27 1.27)) (justify left bottom))
   )
@@
     (effects (font (size 1.27 1.27)) (justify right bottom))
   )
-  (label "IO0_4" (at 199.39 130.81 0)
+  (label "PWM3" (at 77.47 161.29 0)
+    (effects (font (size 1.27 1.27)) (justify left bottom))
+  )
+  (label "IO0_4" (at 199.39 142.24 0)
     (effects (font (size 1.27 1.27)) (justify left bottom))
   )
@@
     (effects (font (size 1.27 1.27)) (justify right bottom))
   )
-  (label "IO1_0" (at 199.39 135.89 0)
+  (label "IO1_0" (at 199.39 125.73 0)
     (effects (font (size 1.27 1.27)) (justify left bottom))
   )
@@
     (effects (font (size 1.27 1.27)) (justify right bottom))
   )
-  (label "PWM10" (at 199.39 67.31 0)
+  (label "PWM6" (at 199.39 67.31 0)
     (effects (font (size 1.27 1.27)) (justify left bottom))
   )
@@
     (effects (font (size 1.27 1.27)) (justify right bottom))
   )
-  (label "PWM14" (at 77.47 171.45 0)
-    (effects (font (size 1.27 1.27)) (justify left bottom))
-  )
   (label "IO0_3" (at 152.4 104.14 180)
     (effects (font (size 1.27 1.27)) (justify right bottom))
@@
     (effects (font (size 1.27 1.27)) (justify right bottom))
   )
-  (label "PWM7" (at 199.39 105.41 0)
+  (label "PWM14" (at 199.39 105.41 0)
     (effects (font (size 1.27 1.27)) (justify left bottom))
   )
@@
     (effects (font (size 1.27 1.27)) (justify right bottom))
   )
-  (label "IO0_3" (at 199.39 128.27 0)
+  (label "IO0_3" (at 199.39 144.78 0)
     (effects (font (size 1.27 1.27)) (justify left bottom))
   )
@@
     (effects (font (size 1.27 1.27)) (justify right bottom))
   )
-  (label "IO0_1" (at 199.39 121.92 0)
-    (effects (font (size 1.27 1.27)) (justify left bottom))
-  )
-  (label "PWM12" (at 77.47 161.29 0)
+  (label "IO0_1" (at 199.39 135.89 0)
     (effects (font (size 1.27 1.27)) (justify left bottom))
   )
@@
     (effects (font (size 1.27 1.27)) (justify right bottom))
   )
-  (label "PWM4" (at 199.39 96.52 0)
-    (effects (font (size 1.27 1.27)) (justify left bottom))
-  )
-  (label "PWM3" (at 199.39 92.71 0)
+  (label "PWM13" (at 199.39 96.52 0)
+    (effects (font (size 1.27 1.27)) (justify left bottom))
+  )
+  (label "PWM10" (at 199.39 92.71 0)
     (effects (font (size 1.27 1.27)) (justify left bottom))
   )
@@
     (effects (font (size 1.27 1.27)) (justify right bottom))
   )
+  (label "PWM0" (at 77.47 176.53 0)
+    (effects (font (size 1.27 1.27)) (justify left bottom))
+  )
   (label "IO1_7" (at 105.41 171.45 180)
     (effects (font (size 1.27 1.27)) (justify right bottom))
@@
     (effects (font (size 1.27 1.27)) (justify right bottom))
   )
-  (label "PWM15" (at 77.47 176.53 0)
-    (effects (font (size 1.27 1.27)) (justify left bottom))
-  )
   (label "AIN5" (at 237.49 147.32 180)
     (effects (font (size 1.27 1.27)) (justify right bottom))
   )
-  (label "PWM2" (at 199.39 90.17 0)
+  (label "PWM11" (at 199.39 90.17 0)
     (effects (font (size 1.27 1.27)) (justify left bottom))
   )
@@
     (effects (font (size 1.27 1.27)) (justify right bottom))
   )
-  (label "IO1_1" (at 199.39 138.43 0)
-    (effects (font (size 1.27 1.27)) (justify left bottom))
-  )
-  (label "PWM6" (at 199.39 102.87 0)
+  (label "IO1_1" (at 199.39 128.27 0)
+    (effects (font (size 1.27 1.27)) (justify left bottom))
+  )
+  (label "PWM15" (at 199.39 102.87 0)
     (effects (font (size 1.27 1.27)) (justify left bottom))
   )
@@
     (effects (font (size 1.27 1.27)) (justify right bottom))
   )
-  (label "PWM8" (at 199.39 62.23 0)
-    (effects (font (size 1.27 1.27)) (justify left bottom))
-  )
+  (label "PWM1" (at 77.47 171.45 0)
+    (effects (font (size 1.27 1.27)) (justify left bottom))
+  )
+  (label "PWM4" (at 199.39 62.23 0)
+    (effects (font (size 1.27 1.27)) (justify left bottom))
+  )
