File: Hardware/Kicad_Project/MASA_Rover_1.0/MASA_Rover_1.0.kicad_sch (KiCad schematic)
At the start: 7 parts, among them J1 Conn_01x04_Female, J2 Conn_02x20_Odd_Even, J3 RJ45

Commit message: update hardware
Connections:
- net +3V3: now also J2.1 (Pin_1); no longer J2.2 (Pin_2)
- net +5V: now also J2.2 (Pin_2), J2.4 (Pin_4); no longer J2.1 (Pin_1), J2.3 (Pin_3)
- net BTN: now also J2.40 (Pin_40); no longer J2.31 (Pin_31)
- net EC11_A: now also J2.18 (Pin_18); no longer J2.17 (Pin_17)
- net EC11_B: now also J2.16 (Pin_16); no longer J2.15 (Pin_15)
- net EC11_SW: now also J2.22 (Pin_22); no longer J2.21 (Pin_21)
- net GND: now also J2.14 (Pin_14), J2.20 (Pin_20), J2.25 (Pin_25), J2.30 (Pin_30), J2.34 (Pin_34), J2.39 (Pin_39), J2.6 (Pin_6), J2.9 (Pin_9); no longer J2.10 (Pin_10), J2.13 (Pin_13), J2.19 (Pin_19), J2.26 (Pin_26), J2.29 (Pin_29), J2.33 (Pin_33), J2.40 (Pin_40), J2.5 (Pin_5)
- net LCD0: now also J2.11 (Pin_11); no longer J2.12 (Pin_12)
- net LCD1: now also J2.13 (Pin_13); no longer J2.14 (Pin_14)
- net LCD2: now also J2.15 (Pin_15); no longer J2.16 (Pin_16)
- net LCD3: now also J2.29 (Pin_29); no longer J2.30 (Pin_30)
- net LCD4: now also J2.31 (Pin_31); no longer J2.32 (Pin_32)
- net LCD5: now also J2.33 (Pin_33); no longer J2.34 (Pin_34)
- net LCD6: now also J2.35 (Pin_35); no longer J2.36 (Pin_36)
- net LCD7: now also J2.37 (Pin_37); no longer J2.38 (Pin_38)
- net LCD_E: now also J2.36 (Pin_36); no longer J2.37 (Pin_37)
- net LCD_RS: now also J2.32 (Pin_32); no longer J2.39 (Pin_39)
- net LCD_RW: now also J2.38 (Pin_38); no longer J2.35 (Pin_35)
- net SCL: now also J2.28 (Pin_28); no longer J2.27 (Pin_27)
- net SDA: now also J2.27 (Pin_27); no longer J2.28 (Pin_28)
- net UART_RXD: now also J2.8 (Pin_8); no longer J2.7 (Pin_7)
- net UART_TXD: now also J2.10 (Pin_10); no longer J2.9 (Pin_9)
