File: Hardware/Kicad_Project/MASA_Rover_1.0/MASA_Rover_1.1.kicad_pcb (KiCad board)
At the start: 4 copper layers, 136 x 100 mm, 196 parts, among them J1 Conn_01x04_Female, J10 Screw_Terminal_01x01, J12 Conn_01x03_Male, J13 Conn_01x03_Male, J14 Conn_01x03_Male, J15 Conn_01x03_Male, J16 Screw_Terminal_01x01, J17 Screw_Terminal_01x01, J18 Screw_Terminal_01x01, J19 Screw_Terminal_01x01, J2 Conn_02x20_Odd_Even, J20 Screw_Terminal_01x01, J21 Screw_Terminal_01x01, J22 Screw_Terminal_01x01, J23 Screw_Terminal_01x01, J24 Screw_Terminal_01x01, J26 Conn_01x04_Male, J27 Conn_01x04_Male, J28 Screw_Terminal_01x01, J29 Screw_Terminal_01x01, J3 RJ45, J4 Screw_Terminal_01x01, J5 Screw_Terminal_01x01, J6 Conn_01x04, J7 Conn_02x10_Top_Bottom, J8 Screw_Terminal_01x01, J9 Screw_Terminal_01x01, Q1 FQD8P10TM, Q10 T2N7002, Q11 T2N7002, Q2 BC847BS, Q3 IRLML0060TRPBF, Q4 T2N7002, Q5 T2N7002, Q6 T2N7002, Q7 T2N7002, Q8 T2N7002, Q9 T2N7002, U1 BCM857BS, U10 DRV8876,16-HTSSOP, U11 DRV8876,16-HTSSOP, U12 DRV8876,16-HTSSOP, U13 DRV8876,16-HTSSOP, U2 MAX20457,28-TQFN, U3 LCD-16X2, U4 MAX11603EEE+, U5 PCA9535D, U6 PCA9685PW_112, U7 LTC6102HVxMS8, U8 LTC6102HVxMS8, U9 LTC6247,8-TSSOP

Commit message: update hardware
Parts:
- added A3: Pololu_Breakout_DRV8825, Module:Pololu_Breakout-16_15.2x20.3mm, F.Cu at (177.2, 67.2)
- added A4: Pololu_Breakout_DRV8825, Module:Pololu_Breakout-16_15.2x20.3mm, F.Cu at (177.2, 88.4)
- added C51: 10u, Capacitor_SMD:C_0805_2012Metric_Pad1.18x1.45mm_HandSolder, F.Cu at (339.3, 98.9)
- added C52: 100n, Capacitor_SMD:C_0805_2012Metric_Pad1.18x1.45mm_HandSolder, F.Cu at (342.4, 73.8)
- added C53: 10u, Capacitor_SMD:C_0805_2012Metric_Pad1.18x1.45mm_HandSolder, F.Cu at (339.3, 95.9)
- added C54: 100n, Capacitor_SMD:C_0805_2012Metric_Pad1.18x1.45mm_HandSolder, F.Cu at (352.2, 90.2)
- added C55: 1u, Capacitor_SMD:C_0805_2012Metric_Pad1.18x1.45mm_HandSolder, F.Cu at (520.8, 99.4)
- added C56: 1u, Capacitor_SMD:C_0805_2012Metric_Pad1.18x1.45mm_HandSolder, F.Cu at (516.0, 99.4)
- added C57: 1u, Capacitor_SMD:C_0805_2012Metric_Pad1.18x1.45mm_HandSolder, F.Cu at (506.5, 120.1)
- added C58: 1u, Capacitor_SMD:C_0805_2012Metric_Pad1.18x1.45mm_HandSolder, F.Cu at (516.0, 102.4)
- added C59: 100n, Capacitor_SMD:C_0805_2012Metric_Pad1.18x1.45mm_HandSolder, B.Cu at (191.2, 123.0)
- added C60: 100n, Capacitor_SMD:C_0805_2012Metric_Pad1.18x1.45mm_HandSolder, B.Cu at (188.1, 124.1)
- added C61: 10u, Capacitor_SMD:C_0805_2012Metric_Pad1.18x1.45mm_HandSolder, B.Cu at (188.1, 121.9)
- added C62: 100n, Capacitor_SMD:C_0805_2012Metric_Pad1.18x1.45mm_HandSolder, F.Cu at (200.3, 133.3)
- added C63: 100n, Capacitor_SMD:C_0805_2012Metric_Pad1.18x1.45mm_HandSolder, F.Cu at (199.2, 136.4)
- added C64: 10u, Capacitor_SMD:C_0805_2012Metric_Pad1.18x1.45mm_HandSolder, F.Cu at (201.4, 136.4)
- added C65: 22n, Capacitor_SMD:C_0805_2012Metric_Pad1.18x1.45mm_HandSolder, B.Cu at (194.3, 124.0)
- added C66: 22n, Capacitor_SMD:C_0805_2012Metric_Pad1.18x1.45mm_HandSolder, F.Cu at (199.3, 130.3)
- added C67: 100n, Capacitor_SMD:C_0805_2012Metric_Pad1.18x1.45mm_HandSolder, B.Cu at (238.3, 122.0)
- added C68: 100n, Capacitor_SMD:C_0805_2012Metric_Pad1.18x1.45mm_HandSolder, B.Cu at (244.0, 128.8)
- added C69: 10u, Capacitor_SMD:C_0805_2012Metric_Pad1.18x1.45mm_HandSolder, B.Cu at (238.5, 125.0)
- added C70: 100n, Capacitor_SMD:C_0805_2012Metric_Pad1.18x1.45mm_HandSolder, F.Cu at (219.1, 132.7)
- added C71: 100n, Capacitor_SMD:C_0805_2012Metric_Pad1.18x1.45mm_HandSolder, F.Cu at (218.0, 135.8)
- added C72: 10u, Capacitor_SMD:C_0805_2012Metric_Pad1.18x1.45mm_HandSolder, F.Cu at (220.2, 135.8)
- added C73: 22n, Capacitor_SMD:C_0805_2012Metric_Pad1.18x1.45mm_HandSolder, B.Cu at (244.0, 125.8)
- added C74: 22n, Capacitor_SMD:C_0805_2012Metric_Pad1.18x1.45mm_HandSolder, F.Cu at (218.2, 129.7)
- added J11: Screw_Terminal_01x01, MASA_footprint:ScrewTerminal_1x01_5x7mm, F.Cu at (129.5, 155.7)
- added J25: Screw_Terminal_01x01, MASA_footprint:ScrewTerminal_1x01_5x7mm, F.Cu at (139.1, 155.8)
- added J30: Screw_Terminal_01x01, MASA_footprint:ScrewTerminal_1x01_5x7mm, F.Cu at (190.9, 59.0)
- added J31: RJ45, Connector_RJ:RJ45_Amphenol_54602-x08_Horizontal, F.Cu at (267.9, 53.8)
- added J32: Conn_01x04, Connector_PinHeader_2.54mm:PinHeader_1x04_P2.54mm_Vertical, F.Cu at (310.1, 79.5)
- added J33: Conn_02x10_Top_Bottom, Connector_PinHeader_2.54mm:PinHeader_2x10_P2.54mm_Vertical, F.Cu at (313.7, 79.5)
- added J34: Screw_Terminal_01x01, MASA_footprint:ScrewTerminal_1x01_5x7mm, F.Cu at (220.7, 57.9)
- added J35: Conn_01x03_Male, Connector_PinHeader_2.54mm:PinHeader_1x03_P2.54mm_Vertical, F.Cu at (515.4, 86.1)
- added J36: Conn_01x03_Male, Connector_PinHeader_2.54mm:PinHeader_1x03_P2.54mm_Vertical, F.Cu at (520.0, 86.1)
- added J37: Conn_01x03_Male, Connector_PinHeader_2.54mm:PinHeader_1x03_P2.54mm_Vertical, F.Cu at (506.4, 97.1)
- added J38: Conn_01x03_Male, Connector_PinHeader_2.54mm:PinHeader_1x03_P2.54mm_Vertical, F.Cu at (506.4, 106.8)
- added J39: Screw_Terminal_01x01, MASA_footprint:ScrewTerminal_1x01_5x7mm, F.Cu at (180.4, 133.8)
- added J40: Screw_Terminal_01x01, MASA_footprint:ScrewTerminal_1x01_5x7mm, F.Cu at (186.7, 142.6)
- added J41: Screw_Terminal_01x01, MASA_footprint:ScrewTerminal_1x01_5x7mm, F.Cu at (180.5, 123.0)
- added J42: Screw_Terminal_01x01, MASA_footprint:ScrewTerminal_1x01_5x7mm, F.Cu at (197.5, 142.6)
- added J43: Screw_Terminal_01x01, MASA_footprint:ScrewTerminal_1x01_5x7mm, F.Cu at (227.6, 133.8)
- added J44: Screw_Terminal_01x01, MASA_footprint:ScrewTerminal_1x01_5x7mm, F.Cu at (210.6, 142.6)
- added J45: Screw_Terminal_01x01, MASA_footprint:ScrewTerminal_1x01_5x7mm, F.Cu at (227.5, 123.0)
- added J46: Screw_Terminal_01x01, MASA_footprint:ScrewTerminal_1x01_5x7mm, F.Cu at (221.3, 142.6)
- added J47: Screw_Terminal_01x01, MASA_footprint:ScrewTerminal_1x01_5x7mm, F.Cu at (220.3, 113.2)
- added J48: Conn_01x04_Male, Connector_PinHeader_2.54mm:PinHeader_1x04_P2.54mm_Vertical, F.Cu at (180.8, 72.1)
- added J49: Conn_01x04_Male, Connector_PinHeader_2.54mm:PinHeader_1x04_P2.54mm_Vertical, F.Cu at (180.5, 93.4)
- added J50: Screw_Terminal_01x01, MASA_footprint:ScrewTerminal_1x01_5x7mm, F.Cu at (187.8, 113.2)
- added JP13: Jumper_3_Bridged12, Jumper:SolderJumper-3_P1.3mm_Bridged12_Pad1.0x1.5mm, F.Cu at (347.0, 90.5)
- added JP14: Jumper_3_Bridged12, Jumper:SolderJumper-3_P1.3mm_Bridged12_Pad1.0x1.5mm, F.Cu at (355.7, 79.3)
- added JP15: Jumper_3_Bridged12, Jumper:SolderJumper-3_P1.3mm_Bridged12_Pad1.0x1.5mm, F.Cu at (334.0, 100.0)
- added JP16: Jumper_3_Bridged12, Jumper:SolderJumper-3_P1.3mm_Bridged12_Pad1.0x1.5mm, F.Cu at (334.0, 96.2)
- added JP17: Jumper_3_Bridged12, Jumper:SolderJumper-3_P1.3mm_Bridged12_Pad1.0x1.5mm, F.Cu at (252.5, 135.6)
- added JP18: Jumper_3_Bridged12, Jumper:SolderJumper-3_P1.3mm_Bridged12_Pad1.0x1.5mm, F.Cu at (197.6, 161.7)
- added JP19: Jumper_3_Open, Jumper:SolderJumper-3_P1.3mm_Open_Pad1.0x1.5mm, F.Cu at (252.5, 138.3)
- added JP20: Jumper_3_Open, Jumper:SolderJumper-3_P1.3mm_Open_Pad1.0x1.5mm, F.Cu at (197.6, 164.4)
- added JP21: Jumper_3_Bridged12, Jumper:SolderJumper-3_P1.3mm_Bridged12_Pad1.0x1.5mm, F.Cu at (351.9, 129.7)
- added JP22: Jumper_3_Bridged12, Jumper:SolderJumper-3_P1.3mm_Bridged12_Pad1.0x1.5mm, F.Cu at (268.5, 162.1)
- added JP23: Jumper_3_Open, Jumper:SolderJumper-3_P1.3mm_Open_Pad1.0x1.5mm, F.Cu at (351.9, 132.4)
- added JP24: Jumper_3_Open, Jumper:SolderJumper-3_P1.3mm_Open_Pad1.0x1.5mm, F.Cu at (268.5, 159.1)
- added Q12: T2N7002, Package_TO_SOT_SMD:SOT-23, F.Cu at (511.2, 104.6)
- added Q13: T2N7002, Package_TO_SOT_SMD:SOT-23, F.Cu at (524.8, 86.0)
- added Q14: T2N7002, Package_TO_SOT_SMD:SOT-23, F.Cu at (515.5, 95.7)
- added Q15: T2N7002, Package_TO_SOT_SMD:SOT-23, F.Cu at (520.4, 95.7)
- added Q16: T2N7002, Package_TO_SOT_SMD:SOT-23, F.Cu at (511.2, 100.1)
- added Q17: T2N7002, Package_TO_SOT_SMD:SOT-23, F.Cu at (524.8, 90.4)
- added Q18: T2N7002, Package_TO_SOT_SMD:SOT-23, F.Cu at (529.7, 86.0)
- added Q19: T2N7002, Package_TO_SOT_SMD:SOT-23, F.Cu at (506.5, 116.4)
- added R54: 10k, Resistor_SMD:R_0805_2012Metric_Pad1.20x1.40mm_HandSolder, F.Cu at (339.2, 101.9)
- added R55: 10k, Resistor_SMD:R_0805_2012Metric_Pad1.20x1.40mm_HandSolder, F.Cu at (360.9, 79.0)
- added R56: 10k, Resistor_SMD:R_0805_2012Metric_Pad1.20x1.40mm_HandSolder, F.Cu at (355.3, 82.8)
- added R57: 100k, Resistor_SMD:R_0805_2012Metric_Pad1.20x1.40mm_HandSolder, F.Cu at (534.5, 85.2)
- added R58: 10k, Resistor_SMD:R_0805_2012Metric_Pad1.20x1.40mm_HandSolder, F.Cu at (525.2, 94.1)
- added R59: 10k, Resistor_SMD:R_0805_2012Metric_Pad1.20x1.40mm_HandSolder, F.Cu at (539.3, 85.2)
- added R60: 100k, Resistor_SMD:R_0805_2012Metric_Pad1.20x1.40mm_HandSolder, F.Cu at (511.3, 111.2)
- added R61: 10k, Resistor_SMD:R_0805_2012Metric_Pad1.20x1.40mm_HandSolder, F.Cu at (534.5, 88.2)
- added R62: 10k, Resistor_SMD:R_0805_2012Metric_Pad1.20x1.40mm_HandSolder, F.Cu at (529.6, 89.7)
- added R63: 100k, Resistor_SMD:R_0805_2012Metric_Pad1.20x1.40mm_HandSolder, F.Cu at (506.4, 123.1)
- added R64: 10k, Resistor_SMD:R_0805_2012Metric_Pad1.20x1.40mm_HandSolder, F.Cu at (525.6, 97.1)
- added R65: 10k, Resistor_SMD:R_0805_2012Metric_Pad1.20x1.40mm_HandSolder, F.Cu at (530.0, 92.6)
- added R66: 100k, Resistor_SMD:R_0805_2012Metric_Pad1.20x1.40mm_HandSolder, F.Cu at (515.8, 108.3)
- added R67: 10k, Resistor_SMD:R_0805_2012Metric_Pad1.20x1.40mm_HandSolder, F.Cu at (511.1, 108.3)
- added R68: 10k, Resistor_SMD:R_0805_2012Metric_Pad1.20x1.40mm_HandSolder, F.Cu at (520.8, 102.4)
- added R69: 100k, Resistor_SMD:R_0805_2012Metric_Pad1.20x1.40mm_HandSolder, B.Cu at (188.1, 136.2)
- added R70: 100k, Resistor_SMD:R_0805_2012Metric_Pad1.20x1.40mm_HandSolder, F.Cu at (187.6, 132.1)
- added R71: 100k, Resistor_SMD:R_0805_2012Metric_Pad1.20x1.40mm_HandSolder, F.Cu at (357.1, 131.4)
- added R72: 100k, Resistor_SMD:R_0805_2012Metric_Pad1.20x1.40mm_HandSolder, F.Cu at (268.5, 164.6)
- added REF**: MountingHole_2.7mm_M2.5, MountingHole:MountingHole_2.7mm_M2.5, F.Cu at (178.0, 55.0)
- added REF**: MountingHole_2.7mm_M2.5, MountingHole:MountingHole_2.7mm_M2.5, F.Cu at (230.0, 55.0)
- added REF**: MountingHole_2.7mm_M2.5, MountingHole:MountingHole_2.7mm_M2.5, F.Cu at (230.0, 145.0)
- added REF**: MountingHole_2.7mm_M2.5, MountingHole:MountingHole_2.7mm_M2.5, F.Cu at (178.0, 145.0)
- added TP10: TestPoint, TestPoint:TestPoint_Pad_D2.0mm, B.Cu at (186.7, 138.9)
- added TP11: TestPoint, TestPoint:TestPoint_Pad_D2.0mm, B.Cu at (186.0, 133.8)
- added TP12: TestPoint, TestPoint:TestPoint_Pad_D2.0mm, F.Cu at (357.5, 128.3)
- added TP13: TestPoint, TestPoint:TestPoint_Pad_D2.0mm, F.Cu at (268.6, 167.3)
- added U14: PCA9535D, Package_SO:SOIC-24W_7.5x15.4mm_P1.27mm, F.Cu at (337.7, 86.0)
- added U15: PCA9685PW_112, Package_SO:TSSOP-28_4.4x9.7mm_P0.65mm, F.Cu at (348.5, 83.1)
- added U16: DRV8876,16-HTSSOP, Package_SO:HTSSOP-16-1EP_4.4x5mm_P0.65mm_EP3.4x5mm, B.Cu at (190.4, 129.5)
- added U17: DRV8876,16-HTSSOP, Package_SO:HTSSOP-16-1EP_4.4x5mm_P0.65mm_EP3.4x5mm, F.Cu at (193.7, 133.9)
- added U18: DRV8876,16-HTSSOP, Package_SO:HTSSOP-16-1EP_4.4x5mm_P0.65mm_EP3.4x5mm, B.Cu at (245.0, 120.0)
- added U19: DRV8876,16-HTSSOP, Package_SO:HTSSOP-16-1EP_4.4x5mm_P0.65mm_EP3.4x5mm, F.Cu at (212.0, 133.3)
- moved REF** 1.75 mm to (152.1, 131.8)
- moved D2 0.15 mm to (146.1, 59.9)
- moved D3 0.12 mm to (148.1, 59.9)
Routing:
- net /Rover Extension/DC Motor Ext./MOT2-: track 0.00 -> 33.2 mm
- net /Rover Extension/DC Motor Ext./MOT3-: track 0.00 -> 30.8 mm
- net /Rover Extension/DC Motor Ext./MOT1-: track 0.00 -> 30.0 mm
- net /Rover Extension/DC Motor Ext./MOT3+: track 0.00 -> 29.4 mm
- net GND2: track 0.00 -> 26.9 mm, vias 0 -> 6
- net /Rover Extension/DC Motor Ext./VCCdc: track 0.00 -> 24.2 mm, vias 0 -> 1
- net /Rover Extension/DC Motor Ext./MOT1+: track 0.00 -> 23.7 mm
- net /Rover Extension/DC Motor Ext./MOT2+: track 0.00 -> 22.0 mm
- net Net-(JP17-Pad2): track 0.00 -> 10.2 mm, vias 0 -> 1
- net +3V3: track 201.6 -> 210.5 mm
- net Net-(R70-Pad2): track 0.00 -> 6.07 mm, vias 0 -> 1
- net Net-(R69-Pad2): track 0.00 -> 6.01 mm
- net Net-(C74-Pad1): track 0.00 -> 5.72 mm
- net Net-(C65-Pad1): track 0.00 -> 5.44 mm
- net Net-(C66-Pad1): track 0.00 -> 5.39 mm
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Other:
- board size 136 x 100 mm -> 200 x 100 mm
- board text removed: "+ -"
- board text removed: "1"
- board text removed: "2"
- board text removed: "3"
- board text removed: "4"
- board text removed: "DC 1"
- board text removed: "DC 2"
- board text removed: "DC 3"
- board text removed: "DC 4"
- board text removed: "GND"
- board text removed: "GND 5V0 SIG"
- board text removed: "MASA rover 1.0"
- board text removed: "Peak Power Measurement"
- board text removed: "Servo"
- board text removed: "VCCdc"
- board text removed: "VCCentre"
- board text removed: "VCCsortie"
- board text removed: "VCCstp"
- board text removed: "by: Yoann Scrosati & Lucas Mongrain"
- board text removed: "extension"
