File: Hardware/Kicad_Project/MASA_Rover_1.0/RoverExtension.kicad_sch (KiCad schematic)
At the start: 17 parts, among them J30 Screw_Terminal_01x01, J31 RJ45, J32 Conn_01x04, J33 Conn_02x10_Top_Bottom, U14 PCA9535D, U15 PCA9685PW_112

Commit message: update hardware
Connections:
- net GND is gone; now on net GND2: C53.2, C54.2
Changed lines of the file:
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@@
-    (pin "1")
-  )
-  (symbol (lib_id "power:GND") (at 96.52 104.14 0) (unit 1)
-    (in_bom yes) (on_board yes) (fields_autoplaced)
-    (property "Reference" "#PWR0189" (id 0) (at 96.52 110.49 0)
-      (effects (font (size 1.27 1.27)) hide)
-    )
-    (property "Value" "GND" (id 1) (at 96.52 108.5834 0))
-    (property "Footprint" "" (id 2) (at 96.52 104.14 0)
-      (effects (font (size 1.27 1.27)) hide)
-    )
-    (property "Datasheet" "" (id 3) (at 96.52 104.14 0)
-      (effects (font (size 1.27 1.27)) hide)
-    )
     (pin "1")
   )
@@
     )
     (property "Datasheet" "" (id 3) (at 59.69 135.89 0)
+      (effects (font (size 1.27 1.27)) hide)
+    )
+    (pin "1")
+  )
+  (symbol (lib_id "power:GND2") (at 96.52 104.14 0) (unit 1)
+    (in_bom yes) (on_board yes) (fields_autoplaced)
+    (property "Reference" "#PWR?" (id 0) (at 96.52 110.49 0)
+      (effects (font (size 1.27 1.27)) hide)
+    )
+    (property "Value" "GND2" (id 1) (at 96.52 108.5834 0))
+    (property "Footprint" "" (id 2) (at 96.52 104.14 0)
+      (effects (font (size 1.27 1.27)) hide)
+    )
+    (property "Datasheet" "" (id 3) (at 96.52 104.14 0)
       (effects (font (size 1.27 1.27)) hide)
     )
@@
     (pin "7")
     (pin "8")
+  )
+  (symbol (lib_id "power:GND2") (at 106.68 104.14 0) (unit 1)
+    (in_bom yes) (on_board yes) (fields_autoplaced)
+    (property "Reference" "#PWR?" (id 0) (at 106.68 110.49 0)
+      (effects (font (size 1.27 1.27)) hide)
+    )
+    (property "Value" "GND2" (id 1) (at 106.68 108.5834 0))
+    (property "Footprint" "" (id 2) (at 106.68 104.14 0)
+      (effects (font (size 1.27 1.27)) hide)
+    )
+    (property "Datasheet" "" (id 3) (at 106.68 104.14 0)
+      (effects (font (size 1.27 1.27)) hide)
+    )
+    (pin "1")
   )
   (symbol (lib_id "Device:R") (at 59.69 50.8 0) (unit 1)
@@
       (effects (font (size 1.27 1.27)) hide)
     )
-    (pin "1")
-  )
-  (symbol (lib_id "power:GND") (at 106.68 104.14 0) (unit 1)
-    (in_bom yes) (on_board yes) (fields_autoplaced)
-    (property "Reference" "#PWR0190" (id 0) (at 106.68 110.49 0)
-      (effects (font (size 1.27 1.27)) hide)
-    )
-    (property "Value" "GND" (id 1) (at 106.68 108.5834 0))
-    (property "Footprint" "" (id 2) (at 106.68 104.14 0)
-      (effects (font (size 1.27 1.27)) hide)
-    )
-    (property "Datasheet" "" (id 3) (at 106.68 104.14 0)
-      (effects (font (size 1.27 1.27)) hide)
-    )
