File: Hardware/Kicad_Project/MASA_Rover_1.0/ServoMotorExt.kicad_sch (KiCad schematic)
At the start: 29 parts, among them J34 Screw_Terminal_01x01, J35 Conn_01x03_Male, J36 Conn_01x03_Male, J37 Conn_01x03_Male, J38 Conn_01x03_Male, Q12 T2N7002, Q13 T2N7002, Q14 T2N7002, Q15 T2N7002, Q16 T2N7002, Q17 T2N7002, Q18 T2N7002, Q19 T2N7002

Commit message: update hardware
Connections:
- net GND is gone; now on net GND2: J35.3 (Pin_3), J36.3 (Pin_3), J37.3 (Pin_3), J38.3 (Pin_3)
Changed lines of the file:
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@@
     (effects (font (size 1.27 1.27)) (justify right))
-  )
-  (symbol (lib_id "power:GND") (at 100.33 111.76 180) (unit 1)
-    (in_bom yes) (on_board yes) (fields_autoplaced)
-    (property "Reference" "#PWR0216" (id 0) (at 100.33 105.41 0)
-      (effects (font (size 1.27 1.27)) hide)
-    )
-    (property "Value" "GND" (id 1) (at 100.33 108.1842 0))
-    (property "Footprint" "" (id 2) (at 100.33 111.76 0)
-      (effects (font (size 1.27 1.27)) hide)
-    )
-    (property "Datasheet" "" (id 3) (at 100.33 111.76 0)
-      (effects (font (size 1.27 1.27)) hide)
-    )
-    (pin "1")
   )
   (symbol (lib_id "Device:R") (at 74.93 143.51 0) (unit 1)
@@
     (pin "1")
   )
-  (symbol (lib_id "power:GND") (at 100.33 149.86 180) (unit 1)
-    (in_bom yes) (on_board yes) (fields_autoplaced)
-    (property "Reference" "#PWR0221" (id 0) (at 100.33 143.51 0)
-      (effects (font (size 1.27 1.27)) hide)
-    )
-    (property "Value" "GND" (id 1) (at 100.33 146.2842 0))
-    (property "Footprint" "" (id 2) (at 100.33 149.86 0)
-      (effects (font (size 1.27 1.27)) hide)
-    )
-    (property "Datasheet" "" (id 3) (at 100.33 149.86 0)
-      (effects (font (size 1.27 1.27)) hide)
-    )
-    (pin "1")
-  )
   (symbol (lib_id "Device:C") (at 106.68 67.31 0) (unit 1)
     (in_bom yes) (on_board yes) (fields_autoplaced)
@@
     (pin "1")
     (pin "2")
-  )
-  (symbol (lib_id "power:GND") (at 100.33 73.66 180) (unit 1)
-    (in_bom yes) (on_board yes) (fields_autoplaced)
-    (property "Reference" "#PWR0211" (id 0) (at 100.33 67.31 0)
-      (effects (font (size 1.27 1.27)) hide)
-    )
-    (property "Value" "GND" (id 1) (at 100.33 70.0842 0))
-    (property "Footprint" "" (id 2) (at 100.33 73.66 0)
-      (effects (font (size 1.27 1.27)) hide)
-    )
-    (property "Datasheet" "" (id 3) (at 100.33 73.66 0)
-      (effects (font (size 1.27 1.27)) hide)
-    )
-    (pin "1")
   )
   (symbol (lib_id "power:GND2") (at 74.93 121.92 0) (unit 1)
@@
     (pin "3")
   )
+  (symbol (lib_id "power:GND2") (at 100.33 35.56 180) (unit 1)
+    (in_bom yes) (on_board yes) (fields_autoplaced)
+    (property "Reference" "#PWR0206" (id 0) (at 100.33 29.21 0)
+      (effects (font (size 1.27 1.27)) hide)
+    )
+    (property "Value" "GND2" (id 1) (at 100.33 31.9842 0))
+    (property "Footprint" "" (id 2) (at 100.33 35.56 0)
+      (effects (font (size 1.27 1.27)) hide)
+    )
+    (property "Datasheet" "" (id 3) (at 100.33 35.56 0)
+      (effects (font (size 1.27 1.27)) hide)
+    )
+    (pin "1")
+  )
   (symbol (lib_id "Device:C") (at 106.68 105.41 0) (unit 1)
     (in_bom yes) (on_board yes) (fields_autoplaced)
@@
     (pin "3")
   )
+  (symbol (lib_id "power:GND2") (at 100.33 73.66 180) (unit 1)
+    (in_bom yes) (on_board yes) (fields_autoplaced)
+    (property "Reference" "#PWR0211" (id 0) (at 100.33 67.31 0)
+      (effects (font (size 1.27 1.27)) hide)
+    )
+    (property "Value" "GND2" (id 1) (at 100.33 70.0842 0))
+    (property "Footprint" "" (id 2) (at 100.33 73.66 0)
+      (effects (font (size 1.27 1.27)) hide)
+    )
+    (property "Datasheet" "" (id 3) (at 100.33 73.66 0)
+      (effects (font (size 1.27 1.27)) hide)
+    )
+    (pin "1")
+  )
   (symbol (lib_id "Device:Q_NMOS_GSD") (at 72.39 76.2 0) (unit 1)
     (in_bom yes) (on_board yes) (fields_autoplaced)
@@
     (pin "1")
   )
+  (symbol (lib_id "power:GND2") (at 100.33 149.86 180) (unit 1)
+    (in_bom yes) (on_board yes) (fields_autoplaced)
+    (property "Reference" "#PWR0216" (id 0) (at 100.33 143.51 0)
+      (effects (font (size 1.27 1.27)) hide)
+    )
+    (property "Value" "GND2" (id 1) (at 100.33 146.2842 0))
+    (property "Footprint" "" (id 2) (at 100.33 149.86 0)
+      (effects (font (size 1.27 1.27)) hide)
+    )
+    (property "Datasheet" "" (id 3) (at 100.33 149.86 0)
+      (effects (font (size 1.27 1.27)) hide)
+    )
+    (pin "1")
+  )
   (symbol (lib_id "Device:R") (at 74.93 67.31 0) (unit 1)
     (in_bom yes) (on_board yes) (fields_autoplaced)
@@
     (pin "1")
     (pin "2")
-  )
-  (symbol (lib_id "power:GND") (at 100.33 35.56 180) (unit 1)
-    (in_bom yes) (on_board yes) (fields_autoplaced)
-    (property "Reference" "#PWR0206" (id 0) (at 100.33 29.21 0)
-      (effects (font (size 1.27 1.27)) hide)
-    )
-    (property "Value" "GND" (id 1) (at 100.33 31.9842 0))
-    (property "Footprint" "" (id 2) (at 100.33 35.56 0)
-      (effects (font (size 1.27 1.27)) hide)
-    )
-    (property "Datasheet" "" (id 3) (at 100.33 35.56 0)
-      (effects (font (size 1.27 1.27)) hide)
-    )
-    (pin "1")
   )
   (symbol (lib_id "Device:R") (at 43.18 118.11 0) (unit 1)
@@
     (pin "2")
   )
+  (symbol (lib_id "power:GND2") (at 100.33 111.76 180) (unit 1)
+    (in_bom yes) (on_board yes) (fields_autoplaced)
+    (property "Reference" "#PWR0221" (id 0) (at 100.33 105.41 0)
+      (effects (font (size 1.27 1.27)) hide)
+    )
+    (property "Value" "GND2" (id 1) (at 100.33 108.1842 0))
+    (property "Footprint" "" (id 2) (at 100.33 111.76 0)
+      (effects (font (size 1.27 1.27)) hide)
+    )
+    (property "Datasheet" "" (id 3) (at 100.33 111.76 0)
+      (effects (font (size 1.27 1.27)) hide)
+    )
+    (pin "1")
+  )
   (symbol (lib_id "Device:Q_NMOS_GSD") (at 52.07 38.1 0) (unit 1)
