File: Hardware/Kicad_Project/MASA_Rover_1.0/UserInterface.kicad_sch (KiCad schematic)
At the start: 14 parts, among them U3 LCD-16X2

Commit message: update hardware
Connections:
- net +3V3: no longer R10.1, R12.1, R9.1
- new net 3V3: R10.1, R12.1, R9.1
Changed lines of the file:
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@@
+    (pin "1")
+  )
+  (symbol (lib_id "tinkerforge:3V3") (at 49.53 34.29 0) (unit 1)
+    (in_bom yes) (on_board yes) (fields_autoplaced)
+    (property "Reference" "#PWR039" (id 0) (at 49.53 38.1 0)
+      (effects (font (size 1.27 1.27)) hide)
+    )
+    (property "Value" "3V3" (id 1) (at 49.53 30.7142 0))
+    (property "Footprint" "" (id 2) (at 49.53 34.29 0))
+    (property "Datasheet" "" (id 3) (at 49.53 34.29 0))
     (pin "1")
   )
@@
     (pin "1")
     (pin "2")
-  )
-  (symbol (lib_id "power:+3V3") (at 91.44 34.29 0) (unit 1)
-    (in_bom yes) (on_board yes) (fields_autoplaced)
-    (property "Reference" "#PWR?" (id 0) (at 91.44 38.1 0)
-      (effects (font (size 1.27 1.27)) hide)
-    )
-    (property "Value" "+3V3" (id 1) (at 91.44 30.7142 0))
-    (property "Footprint" "" (id 2) (at 91.44 34.29 0)
-      (effects (font (size 1.27 1.27)) hide)
-    )
-    (property "Datasheet" "" (id 3) (at 91.44 34.29 0)
-      (effects (font (size 1.27 1.27)) hide)
-    )
-    (pin "1")
   )
   (symbol (lib_id "power:GND") (at 67.31 106.68 0) (unit 1)
@@
     (pin "1")
     (pin "2")
-  )
-  (symbol (lib_id "power:+3V3") (at 60.96 34.29 0) (unit 1)
-    (in_bom yes) (on_board yes) (fields_autoplaced)
-    (property "Reference" "#PWR?" (id 0) (at 60.96 38.1 0)
-      (effects (font (size 1.27 1.27)) hide)
-    )
-    (property "Value" "+3V3" (id 1) (at 60.96 30.7142 0))
-    (property "Footprint" "" (id 2) (at 60.96 34.29 0)
-      (effects (font (size 1.27 1.27)) hide)
-    )
-    (property "Datasheet" "" (id 3) (at 60.96 34.29 0)
-      (effects (font (size 1.27 1.27)) hide)
-    )
-    (pin "1")
   )
   (symbol (lib_id "dk_Encoders:PEC11R-4215F-S0024") (at 83.82 46.99 0) (unit 1)
@@
     (pin "2")
   )
+  (symbol (lib_id "tinkerforge:3V3") (at 91.44 34.29 0) (unit 1)
+    (in_bom yes) (on_board yes) (fields_autoplaced)
+    (property "Reference" "#PWR042" (id 0) (at 91.44 38.1 0)
+      (effects (font (size 1.27 1.27)) hide)
+    )
+    (property "Value" "3V3" (id 1) (at 91.44 30.7142 0))
+    (property "Footprint" "" (id 2) (at 91.44 34.29 0))
+    (property "Datasheet" "" (id 3) (at 91.44 34.29 0))
+    (pin "1")
+  )
   (symbol (lib_id "power:GND") (at 58.42 106.68 0) (unit 1)
     (in_bom yes) (on_board yes) (fields_autoplaced)
@@
     )
     (property "Datasheet" "" (id 3) (at 58.42 106.68 0)
-      (effects (font (size 1.27 1.27)) hide)
-    )
-    (pin "1")
-  )
-  (symbol (lib_id "power:+3V3") (at 49.53 34.29 0) (unit 1)
-    (in_bom yes) (on_board yes) (fields_autoplaced)
-    (property "Reference" "#PWR?" (id 0) (at 49.53 38.1 0)
-      (effects (font (size 1.27 1.27)) hide)
-    )
-    (property "Value" "+3V3" (id 1) (at 49.53 30.7142 0))
-    (property "Footprint" "" (id 2) (at 49.53 34.29 0)
-      (effects (font (size 1.27 1.27)) hide)
-    )
-    (property "Datasheet" "" (id 3) (at 49.53 34.29 0)
       (effects (font (size 1.27 1.27)) hide)
     )
@@
     (pin "2")
   )
+  (symbol (lib_id "tinkerforge:3V3") (at 60.96 34.29 0) (unit 1)
+    (in_bom yes) (on_board yes) (fields_autoplaced)
+    (property "Reference" "#PWR040" (id 0) (at 60.96 38.1 0)
+      (effects (font (size 1.27 1.27)) hide)
+    )
+    (property "Value" "3V3" (id 1) (at 60.96 30.7142 0))
+    (property "Footprint" "" (id 2) (at 60.96 34.29 0))
+    (property "Datasheet" "" (id 3) (at 60.96 34.29 0))
+    (pin "1")
+  )
   (symbol (lib_id "power:+3V3") (at 95.25 90.17 0) (unit 1)
